File: board/fpgaboy.sch (KiCad schematic (older format))
At the start: 89 parts, among them J2 Conn_01x06, J4 Conn_01x06, P1 ILI9341, P2 CONN_01X02, P3 USB_OTG, P4 CONN_01X02, Q1 BSS816NW, U2 DSC60XX, U3 GS74116AGP/, U4 BQ21040, U5 NCP1532

Commit message: Board rev B: add QFN 20 weird corner footprint for CP2102N and SOD-923 for TVS diodes. Add TVS and some pullups etc to the schematic.
Parts:
- removed U? (x2): 74LVC2G04, symbol 74xGxx:74LVC2G04
- added C3, C5: 1u, Capacitor_SMD:C_0603_1608Metric, symbol Device:C_Small
- added D3, D4, D5: DF2B7AFS, fpgaboy_parts:SOD-923, symbol Device:D_TVS
- added R25, R26: 220, Resistor_SMD:R_0603_1608Metric, symbol fpgaboy-rescue:R
- added R7, R8: 10, Resistor_SMD:R_0603_1608Metric, symbol Device:R_Small
- added RN2: 10k, fpgaboy_parts:RN4-1206, symbol Device:R_Pack04
- added U8: 74LVC2G04, symbol fpgaboy_parts:74LVC2G04
- C31, C32: renamed from C?; footprint (none) -> Capacitor_SMD:C_0603_1608Metric
- J1: renamed from J?; footprint (none) -> Connector_PinSocket_2.54mm:PinSocket_1x10_P2.54mm_Vertical
- R12: renamed from R?; value 22k -> 100k
- R16: value NF -> 100k
- R21: renamed from R?; value 47k -> 100k
- R23, R24: renamed from R?; footprint (none) -> Resistor_SMD:R_0603_1608Metric
- RN1: renamed from RN?; footprint (none) -> fpgaboy_parts:RN4-1206
- SW1: renamed from SW?; footprint (none) -> Connector_PinSocket_2.54mm:PinSocket_2x01_P2.54mm_Vertical
- U1: renamed from U?; footprint (none) -> Package_QFP:TQFP-144_20x20mm_P0.5mm
- U7: renamed from U?; footprint (none) -> fpgaboy_parts:QFN-20-CORNER
- gave numbers to parts that had none: 7
Connections:
- net uC_~RST is gone; now on net FPGA_~RST: U5.8 (~POR)
- net +1V2: now also U1.111 (VCC[4]), U1.27 (VCC[4]), U1.40 (VCC[4]), U1.92 (VCC[4]), R7.2, R8.2
- net +3V3: now also U1.108 (VPP_2V5), U1.72 (VCC_SPI), RN2.5 (R4.2), RN2.6 (R3.2), RN2.7 (R2.2), RN2.8 (R1.2), U8.5 (VCC); no longer U1.71 (IOB_108_SS)
- net +5V: now also R16.1, D5.2 (A2)
- net AUDIO_PWM: now also U1.83 (IOR_119); no longer U1.80 (IOR_116)
- net CLK_OSC: now also U1.93 (IOR_140_GBIN3); no longer U1.91 (IOR_139)
- net FLASH_IO2: now also U1.61 (IOB_96); no longer U1.60 (IOB_95)
- net FLASH_IO3: now also U1.62 (IOB_102); no longer U1.61 (IOB_96)
- net FLASH_MISO: now also U1.68 (IOB_106_SDI); no longer U1.67 (IOB_105_SDO), U7.19 (RXT/GPIO3)
- net FLASH_MOSI: now also U1.67 (IOB_105_SDO); no longer U1.72 (VCC_SPI)
- net FLASH_SCK: now also U1.70 (IOB_107_SCK); no longer U1.68 (IOB_106_SDI), U7.20 (TXT/GPIO2)
- net FLASH_~CS: now also U1.71 (IOB_108_SS); no longer U1.70 (IOB_107_SCK), U7.1 (RS485/GPIO1)
- net FPGA_CFG_DONE: now also U1.65 (CDONE), RN2.1 (R1.1); no longer U1.46 (VCCIO_2[2]), U1.57 (VCCIO_2[2])
- net FPGA_UART_RX: now also U1.64 (IOB_104_CBSEL1), R25.1; no longer U7.18 (TXD)
- net FPGA_UART_TX: now also U1.63 (IOB_103_CBSEL0), R26.1, RN2.3 (R3.1); no longer U7.17 (RXD)
- net GND: now also U1.103 (GND[9]), U1.13 (GND[9]), U1.132 (GND[9]), U1.14 (GND[9]), U1.140 (GND[9]), U1.5 (GND[9]), U1.59 (GND[9]), U1.69 (GND[9]), U1.86 (GND[9]), D3.1 (A1), D4.1 (A1), D5.1 (A1), U8.2 (GND); no longer R16.2
- net GPIO_SW0: now also U1.37 (IOB_56)
- net GPIO_SW1: now also U1.38 (IOB_57)
- net GPIO_SW2: now also U1.39 (IOB_61)
- net GPIO_SW3: now also U1.41 (IOB_63)
- net GPIO_SW4: now also U1.42 (IOB_64)
- net GPIO_SW5: now also U1.43 (IOB_71)
- net GPIO_SW6: now also U1.44 (IOB_72)
- net GPIO_SW7: now also U1.45 (IOB_73)
- net GPIO_SW8: now also U1.47 (IOB_79)
- net GPIO_SW9: now also U1.48 (IOB_80)
- net LCD_CS: now also U1.76 (IOR_112); no longer U1.75 (IOR_111)
- net LCD_D~C~: now also U1.78 (IOR_114); no longer U1.76 (IOR_112)
- net LCD_PWM: now also U1.80 (IOR_116); no longer U1.79 (IOR_115)
- net LCD_RESET: now also U1.73 (IOR_109); no longer U1.100 (VCCIO_1[2]), U1.89 (VCCIO_1[2])
- net LCD_SCL: now also U1.79 (IOR_115); no longer U1.78 (IOR_114)
- net LCD_SDA: now also U1.75 (IOR_111); no longer U1.74 (IOR_110)
- net LCD_SDO: now also U1.74 (IOR_110); no longer U1.73 (IOR_109)
- net PWR_EN: now also U8.4
- net USB_DM: now also D4.2 (A2)
- net USB_DP: now also D3.2 (A2)
- net at P3.4 (ID): no longer R16.1
- net at U1.126 (VCCPLL1): now also C3.1, R7.1
- net at U1.127 (GNDPLL1): now also C3.2
- net at U1.53 (GNDPLL0): now also C5.2
- net at U1.54 (VCCPLL0): now also C5.1, R8.1
- net FPGA_~RST: now reaches U1.66 (CRESET_B)
- net FPGA_~RST: now also J1.7 (Pin_7), RN2.2 (R2.1)
- net at C32.1, R24.1, SW1.2: now also U8.1
- net at R23.2: now also U8.3, U8.6
- net at R12.2, R21.1, U7.8 (VBUS): now also R16.2
- removed net FPGA_CFG_~RST: J1.7 (Pin_7), U1.65 (CDONE), U7.2 (CLK/GPIO0)
- new net: U1.100 (VCCIO_1[2]), U1.89 (VCCIO_1[2])
- new net: U1.46 (VCCIO_2[2]), U1.57 (VCCIO_2[2])
- new net: R26.2, U7.17 (RXD)
- new net: R25.2, U7.18 (TXD)
- no-connect marks 10 -> 16
Other:
- note added: "IS61WV25616EDBLL works too"
- note added: "PLL grounds are tied internally,\nshould NOT be connected to board GND"
- note added: "TODO: is it possible to tie VBUS\ndetect to VDD (LDO output)"
- note removed: "Separate nets from 1V2\ndue to RC filter. Must\nexplicitly mark as powered."
- note removed: "TODO: Can we do some nasty bitbashing\nwith these for direct FPGA config?\nAt the very least it's nice to be able\nto reset the FPGA on connect for DFU mode"
- moved on the sheet: C10, C11, C12, C13, C15, C16, C17, C18, C19, C21, C23, C4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
