File: board/riscboy_revb0/riscboy.kicad_pcb (KiCad board)
At the start: 0 parts

Commit message: Start drawing board outline
Parts:
- added REF**: MH_5mm, riscboy:MH_5mm, F.Cu at (166.2, 89.8)
- added REF**: MH_5mm, riscboy:MH_5mm, F.Cu at (104.9, 34.9)
- added REF**: MH_5mm, riscboy:MH_5mm, F.Cu at (105.0, 89.8)
- added REF**: MH_5mm, riscboy:MH_5mm, F.Cu at (166.2, 33.7)
- added REF**: MH_2.5mm, riscboy:MH_2.5mm, F.Cu at (135.2, 106.7)
Other:
- board outline added: 70.3 x 102.1 mm
- copper layers 0 -> 2
Changed lines of the file:
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@@
-(kicad_pcb (version 20210126) (generator pcbnew)
+(kicad_pcb (version 20210228) (generator pcbnew)
+  (general
+    (thickness 1.6)
+  )
+  (paper "A4")
+  (layers
+    (0 "F.Cu" signal)
+    (31 "B.Cu" signal)
+    (32 "B.Adhes" user "B.Adhesive")
+    (33 "F.Adhes" user "F.Adhesive")
+    (34 "B.Paste" user)
+    (35 "F.Paste" user)
+    (36 "B.SilkS" user "B.Silkscreen")
+    (37 "F.SilkS" user "F.Silkscreen")
+    (38 "B.Mask" user)
+    (39 "F.Mask" user)
+    (40 "Dwgs.User" user "User.Drawings")
+    (41 "Cmts.User" user "User.Comments")
+    (42 "Eco1.User" user "User.Eco1")
+    (43 "Eco2.User" user "User.Eco2")
+    (44 "Edge.Cuts" user)
+    (45 "Margin" user)
+    (46 "B.CrtYd" user "B.Courtyard")
+    (47 "F.CrtYd" user "F.Courtyard")
+    (48 "B.Fab" user)
+    (49 "F.Fab" user)
+    (50 "User.1" user)
+    (51 "User.2" user)
+    (52 "User.3" user)
+    (53 "User.4" user)
+    (54 "User.5" user)
+    (55 "User.6" user)
+    (56 "User.7" user)
+    (57 "User.8" user)
+    (58 "User.9" user)
+  )
+  (setup
+    (pad_to_mask_clearance 0)
+    (pcbplotparams
+      (layerselection 0x00010fc_ffffffff)
+      (disableapertmacros false)
+      (usegerberextensions false)
+      (usegerberattributes true)
+      (usegerberadvancedattributes true)
+      (creategerberjobfile true)
+      (svguseinch false)
+      (svgprecision 6)
+      (excludeedgelayer true)
+      (plotframeref false)
+      (viasonmask false)
+      (mode 1)
+      (useauxorigin false)
+      (hpglpennumber 1)
+      (hpglpenspeed 20)
+      (hpglpendiameter 15.000000)
+      (dxfpolygonmode true)
+      (dxfimperialunits true)
+      (dxfusepcbnewfont true)
+      (psnegative false)
+      (psa4output false)
+      (plotreference true)
+      (plotvalue true)
+      (plotinvisibletext false)
+      (sketchpadsonfab false)
+      (subtractmaskfromsilk false)
+      (outputformat 1)
+      (mirror false)
+      (drillshape 1)
+      (scaleselection 1)
+      (outputdirectory "")
+    )
+  )
+  (net 0 "")
+  (footprint "riscboy:MH_5mm" (layer "F.Cu")
+    (at 166.2 89.8)
+    (fp_text reference "REF**" (at 0 -0.5 unlocked) (layer "F.SilkS") hide
+      (effects (font (size 1 1) (thickness 0.15)))
+    )
+    (fp_text value "MH_5mm" (at 0 1 unlocked) (layer "F.Fab")
+      (effects (font (size 1 1) (thickness 0.15)))
+    )
+    (fp_text user "${REFERENCE}" (at 0 2.5 unlocked) (layer "F.Fab")
+      (effects (font (size 1 1) (thickness 0.15)))
+    )
+    (pad "" np_thru_hole circle (at 0 0) (locked) (size 5 5) (drill 5) (layers F&B.Cu *.Mask)
+      (solder_mask_margin 0.3) (clearance 0.4))
+  )
+  (footprint "riscboy:MH_5mm" (layer "F.Cu")
+    (at 104.9 34.9)
+    (fp_text reference "REF**" (at 0 -0.5 unlocked) (layer "F.SilkS") hide
+      (effects (font (size 1 1) (thickness 0.15)))
+    )
+    (fp_text value "MH_5mm" (at 0 1 unlocked) (layer "F.Fab")
+      (effects (font (size 1 1) (thickness 0.15)))
+    )
+    (fp_text user "${REFERENCE}" (at 0 2.5 unlocked) (layer "F.Fab")
+      (effects (font (size 1 1) (thickness 0.15)))
+    )
+    (pad "" np_thru_hole circle (at 0 0) (locked) (size 5 5) (drill 5) (layers F&B.Cu *.Mask)
+      (solder_mask_margin 0.3) (clearance 0.4))
+  )
+  (footprint "riscboy:MH_5mm" (layer "F.Cu")
+    (at 105 89.8)
+    (fp_text reference "REF**" (at 0 -0.5 unlocked) (layer "F.SilkS") hide
+      (effects (font (size 1 1) (thickness 0.15)))
+    )
+    (fp_text value "MH_5mm" (at 0 1 unlocked) (layer "F.Fab")
+      (effects (font (size 1 1) (thickness 0.15)))
+    )
+    (fp_text user "${REFERENCE}" (at 0 2.5 unlocked) (layer "F.Fab")
+      (effects (font (size 1 1) (thickness 0.15)))
+    )
+    (pad "" np_thru_hole circle (at 0 0) (locked) (size 5 5) (drill 5) (layers F&B.Cu *.Mask)
+      (solder_mask_margin 0.3) (clearance 0.4))
+  )
+  (footprint "riscboy:MH_5mm" (layer "F.Cu")
+    (at 166.2 33.7)
+    (fp_text reference "REF**" (at 0 -0.5 unlocked) (layer "F.SilkS") hide
+      (effects (font (size 1 1) (thickness 0.15)))
+    )
+    (fp_text value "MH_5mm" (at 0 1 unlocked) (layer "F.Fab")
+      (effects (font (size 1 1) (thickness 0.15)))
+    )
+    (fp_text user "${REFERENCE}" (at 0 2.5 unlocked) (layer "F.Fab")
+      (effects (font (size 1 1) (thickness 0.15)))
+    )
+    (pad "" np_thru_hole circle (at 0 0) (locked) (size 5 5) (drill 5) (layers F&B.Cu *.Mask)
+      (solder_mask_margin 0.3) (clearance 0.4))
+  )
+  (footprint "riscboy:MH_2.5mm" locked (layer "F.Cu")
+    (at 135.15 106.7)
+    (fp_text reference "REF**" (at 0 -0.5 unlocked) (layer "F.SilkS") hide
+      (effects (font (size 1 1) (thickness 0.15)))
+    )
+    (fp_text value "MH_2.5mm" (at 0 1 unlocked) (layer "F.Fab")
+      (effects (font (size 1 1) (thickness 0.15)))
+    )
+    (fp_text user "${REFERENCE}" (at 0 2.5 unlocked) (layer "F.Fab")
+      (effects (font (size 1 1) (thickness 0.15)))
+    )
+    (pad "" np_thru_hole circle (at 0 0) (locked) (size 2.5 2.5) (drill 2.5) (layers F&B.Cu *.Mask)
+      (solder_mask_margin 1.1) (clearance 1.2))
+  )
+  (gr_arc (start 102 129.2) (end 102 131.2) (angle 90) (layer "Edge.Cuts") (width 0.05))
+  (gr_line (start 139.3 29.1) (end 142.1 31.9) (layer "Edge.Cuts") (width 0.05))
+  (gr_line (start 168.3 30) (end 165 30) (layer "Edge.Cuts") (width 0.05))
+  (gr_line (start 100 129.2) (end 100 32) (layer "Edge.Cuts") (width 0.05))
+  (gr_line (start 109.5 31.3) (end 111 31.3) (layer "Edge.Cuts") (width 0.05))
+  (gr_line (start 142.1 31.9) (end 163.1 31.9) (layer "Edge.Cuts") (width 0.05))
+  (gr_line (start 149 131.2) (end 102 131.2) (layer "Edge.Cuts") (width 0.05))
+  (gr_arc (start 163 131.2) (end 149 131.2) (angle 90) (layer "Edge.Cuts") (width 0.05))
+  (gr_line (start 131 29.1) (end 128.8 31.3) (layer "Edge.Cuts") (width 0.05))
+  (gr_line (start 109.5 30) (end 109.5 31.3) (layer "Edge.Cuts") (width 0.05))
+  (gr_line (start 128.8 31.3) (end 126 31.3) (layer "Edge.Cuts") (width 0.05))
+  (gr_arc (start 168.3 32) (end 170.3 32) (angle -90) (layer "Edge.Cuts") (width 0.05))
+  (gr_arc (start 102 32) (end 100 32) (angle 90) (layer "Edge.Cuts") (width 0.05))
+  (gr_line (start 170.3 32) (end 170.3 117.2) (layer "Edge.Cuts") (width 0.05))
+  (gr_line (start 111 31.3) (end 111 30) (layer "Edge.Cuts") (width 0.05))
+  (gr_line (start 126 30) (end 126 31.3) (layer "Edge.Cuts") (width 0.05))
+  (gr_line (start 165 30) (end 163.1 31.9) (layer "Edge.Cuts") (width 0.05))
+  (gr_line (start 102 30) (end 109.5 30) (layer "Edge.Cuts") (width 0.05))
+  (gr_line (start 111 30) (end 126 30) (layer "Edge.Cuts") (width 0.05))
+  (gr_line (start 139.3 29.1) (end 131 29.1) (layer "Edge.Cuts") (width 0.05))
+  (gr_line (start 163 117.2) (end 170.3 117.2) (layer "Edge.Cuts") (width 0.05))
+  (gr_circle (center 104.9 34.9) (end 107.4 34.9) (layer "User.1") (width 0.1) (fill none))
+  (gr_circle (center 105 89.8) (end 107.5 89.8) (layer "User.1") (width 0.1) (fill none))
+  (gr_circle (center 166.2 89.8) (end 168.7 89.8) (layer "User.1") (width 0.1) (fill none))
+  (gr_circle (center 166.2 33.7) (end 168.7 33.7) (layer "User.1") (width 0.1) (fill none))
+  (gr_circle (center 135.15 106.7) (end 136.4 106.7) (layer "User.1") (width 0.1) (fill none))
 )
